Commit message: laser_link x offsetini düzelt, gps_filter filter host'unu localhost yap
Lidar laser_link origin x=0.5'ten 0.7'ye güncellendi. gps_filter.json'daki
filter servisi host'u 10.10.10.117 yerine localhost olarak düzeltildi;
filter servisi gerçekte brain üzerinde localhost'ta çalışıyor, eski IP
ile /state mesajları hiç gelmiyordu (bu yüzden /rtk/odom yayınlanmıyordu).

Co-Authored-By: Claude Sonnet 4.6 <noreply@anthropic.com>

File: ros2_amiga_ws/amiga_description/urdf/amiga.urdf.xacro (robot description, xacro)
@@ -91,5 +91,5 @@
     <parent link="base_link"/>
     <child link="laser_link"/>
-    <origin rpy="0 0 0" xyz="0.5 0 0.4"/>
+    <origin rpy="0 0 0" xyz="0.7 0 0.4"/>
   </joint>
 </robot>

Commit message: DDS unicast peer-list robot tarafından geri alındı, lidar yönü düzeltildi
FASTRTPS_DEFAULT_PROFILES_FILE'ı robot container'ına eklemek hataydı:
robotun kendi node'ları arası iletişim zaten localhost üzerinden
sorunsuz çalışıyordu (multicast sorunu sadece WiFi üzerinden PC'nin
robotu keşfetmesiyle ilgiliydi). Bu profil robotta tüm node'ların DDS
iletişimini bozdu ("sequence size exceeds remaining buffer" hatalarıyla
ekf/lidar/nav2/robot_state_publisher hiç ayağa kalkamadı). Robot,
default (multicast) discovery'sine geri döndürüldü; unicast peer-list
sadece PC tarafında kullanılacak — PC'nin gönderdiği unicast SPDP
paketini robot normal şekilde yanıtlayacağı için robot tarafında
değişiklik gerekmiyor.

Ayrıca: LiDAR fiziksel olarak 180° ters monte edilmiş, laser_joint
yaw'ı pi olarak düzeltildi.

Co-Authored-By: Claude Sonnet 4.6 <noreply@anthropic.com>

File: ros2_amiga_ws/amiga_description/urdf/amiga.urdf.xacro (robot description, xacro)
@@ -91,5 +91,7 @@
     <parent link="base_link"/>
     <child link="laser_link"/>
-    <origin rpy="0 0 0" xyz="0.7 0 0.4"/>
+    <!-- LiDAR fiziksel olarak 180° ters monte edilmiş; sensörün 0° yönü
+         robotun arkasını gösteriyordu, burada düzeltildi. -->
+    <origin rpy="0 0 ${pi}" xyz="0.7 0 0.4"/>
   </joint>
 </robot>
